Commit message: update manage_mission: done

File: src/lower_layer_mvibot/urdf/fcr.urdf (robot description, URDF)
Before this commit: robot mvibot, 8 links, 7 joints
Joints:
- removed joint $(arg mvibot_seri)/base_link
- removed joint camera1_$(arg mvibot_seri)
- removed joint camera2_$(arg mvibot_seri)
- added joint base_joint: type fixed, parent $(arg mvibot_seri)/base_footprint, child $(arg mvibot_seri)/base_link, origin xyz=0 0.0 0 rpy=0 0 0
- added joint camera1: type fixed, parent $(arg mvibot_seri)/base_link, child camera1_$(arg mvibot_seri), origin xyz=0.438 -0.126 0.411 rpy=${-pi/2} 0 ${pi/9}
- added joint camera2: type fixed, parent $(arg mvibot_seri)/base_link, child camera2_$(arg mvibot_seri), origin xyz=0.438 0.126 0.411 rpy=${-pi/2} 0 ${-pi/9}
